File: Eagle/Bitcrusher.brd (EAGLE design)
At the start: 80 x 100 mm, 18 parts, among them IC1 TL074P, IC2 NE555, Q1 BF245

Commit message: Made eagle schematic more readable.
Routing:
- net N$13: track 47.7 -> 19.1 mm
- net N$10: track 250.5 -> 234.5 mm
- net N$14: track 67.2 -> 57.0 mm
- net N$5: track 18.6 -> 14.3 mm
- net N$6: track 3.07 -> 0.00 mm
- net N$12: track 94.2 -> 91.6 mm
